File: baromodule/rocket_project.kicad_pcb (KiCad board)
At the start: 4 copper layers, 49.9 x 49.9 mm, 27 parts, among them J1 Conn_01x05_MountingPin, J2 Conn_01x04, J3 Conn_01x02_MountingPin, U1 MPXHZ6130, U2 AMS1117-5.0, U3 SHT1x, U4 AMS1117-3.3

Commit message: final
Other:
- board text added: "3.3V GND SCL SDA"
- board text added: "5V"
- board text added: "GND"
- board text added: "GND SCL SDA BARO_dev BARO_raw"
Changed lines of the file:
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@@
 			(plot_on_all_layers_selection 0x0000000_00000000)
 			(disableapertmacros no)
-			(usegerberextensions no)
-			(usegerberattributes yes)
-			(usegerberadvancedattributes yes)
-			(creategerberjobfile yes)
+			(usegerberextensions yes)
+			(usegerberattributes no)
+			(usegerberadvancedattributes no)
+			(creategerberjobfile no)
 			(dashed_line_dash_ratio 12.000000)
 			(dashed_line_gap_ratio 3.000000)
 			(svgprecision 4)
 			(plotframeref no)
-			(viasonmask no)
+			(viasonmask yes)
 			(mode 1)
 			(useauxorigin no)
@@
 			(psa4output no)
 			(plotreference yes)
-			(plotvalue yes)
+			(plotvalue no)
 			(plotfptext yes)
 			(plotinvisibletext no)
 			(sketchpadsonfab no)
-			(subtractmaskfromsilk no)
+			(subtractmaskfromsilk yes)
 			(outputformat 1)
 			(mirror no)
-			(drillshape 1)
+			(drillshape 0)
 			(scaleselection 1)
-			(outputdirectory "")
+			(outputdirectory "gerbers/")
 		)
 	)
@@
 		(tags "connector JST GH horizontal")
 		(property "Reference" "J1"
-			(at 0 -3.899999 270)
+			(at 0 -3.899999 -90)
 			(layer "F.SilkS")
 			(hide yes)
@@
 		)
 		(property "Value" "Conn_01x05_MountingPin"
-			(at 0 3.899999 270)
+			(at 0 3.899999 -90)
 			(layer "F.Fab")
 			(effects
@@
 		)
 		(fp_text user "${REFERENCE}"
-			(at 0 0 270)
+			(at 0 0 -90)
 			(layer "F.Fab")
 			(effects
@@
 		)
 		(property "Value" "22uF"
-			(at 0 1.679999 270)
+			(at 0 1.679999 -90)
 			(layer "F.Fab")
 			(effects
@@
 		)
 		(fp_text user "${REFERENCE}"
-			(at 0 0 270)
+			(at 0 0 -90)
 			(layer "F.Fab")
 			(effects
@@
 		(tags "CMS SOT")
 		(property "Reference" "U2"
-			(at -3.5 -4.500001 360)
+			(at -3.5 -4.500001 0)
 			(layer "F.SilkS")
 			(effects
@@
 		)
 		(property "Value" "AMS1117-5.0"
-			(at 0 4.500001 360)
+			(at 0 4.500001 0)
 			(layer "F.Fab")
 			(effects
@@
 		(tags "resistor handsolder")
 		(property "Reference" "R2"
-			(at -2.75 0 270)
+			(at -2.75 -0.2 -90)
 			(layer "F.SilkS")
 			(effects
@@
 		)
 		(property "Value" "170"
-			(at 0 1.43 270)
+			(at 0 1.43 -90)
 			(layer "F.Fab")
 			(effects
@@
 		)
 		(fp_text user "${REFERENCE}"
-			(at 0 0 270)
+			(at 0 0 -90)
 			(layer "F.Fab")
 			(effects
@@
 		(tags "capacitor")
 		(property "Reference" "C1"
-			(at 0 -1.43 270)
+			(at 0 -1.43 -90)
 			(layer "F.SilkS")
 			(effects
@@
 		)
 		(property "Value" "100n"
-			(at 0 1.43 270)
+			(at 0 1.43 -90)
 			(layer "F.Fab")
 			(effects
@@
 		)
 		(fp_text user "${REFERENCE}"
-			(at 0 0 270)
+			(at 0 0 -90)
 			(layer "F.Fab")
 			(effects
@@
 		(tags "resistor handsolder")
 		(property "Reference" "R3"
-			(at 2.75 0 90)
+			(at 2.8 0.4 90)
 			(layer "F.SilkS")
 			(effects
@@
 		(tags "resistor handsolder")
 		(property "Reference" "R1"
-			(at -2.75 0 270)
+			(at -2.75 0 -90)
 			(layer "F.SilkS")
 			(effects
@@
 		)
 		(property "Value" "51k"
-			(at 0 1.43 270)
+			(at 0 1.43 -90)
 			(layer "F.Fab")
 			(effects
@@
 		)
 		(fp_text user "${REFERENCE}"
-			(at 0 0 270)
+			(at 0 0 -90)
 			(layer "F.Fab")
 			(effects
@@
 		(tags "capacitor")
 		(property "Reference" "C3"
-			(at 2.75 0 360)
+			(at 2.75 0 0)
 			(layer "F.SilkS")
 			(effects
@@
 		)
 		(property "Value" "22uF"
-			(at 0 1.679999 360)
+			(at 0 1.679999 0)
 			(layer "F.Fab")
 			(effects
@@
 		)
 		(fp_text user "${REFERENCE}"
-			(at 0 0 360)
+			(at 0 0 0)
 			(layer "F.Fab")
 			(effects
@@
 		(tags "LED")
 		(property "Reference" "D3"
-			(at -1.6 -1.5 270)
+			(at -1.6 -1.5 -90)
 			(layer "F.SilkS")
 			(effects
@@
 		)
 		(property "Value" "BLU"
-			(at 0 1.43 270)
+			(at 0 1.43 -90)
 			(layer "F.Fab")
 			(effects
@@
 		)
 		(fp_text user "${REFERENCE}"
-			(at 0 0 270)
+			(at 0 0 -90)
 			(layer "F.Fab")
 			(effects
@@
 		(tags "LED")
 		(property "Reference" "D2"
-			(at -1.625 -1.499999 270)
+			(at -1.625 -1.499999 -90)
 			(layer "F.SilkS")
 			(effects
@@
 		)
 		(property "Value" "BLU"
-			(at 0 1.43 270)
+			(at 0 1.43 -90)
 			(layer "F.Fab")
 			(effects
@@
 		)
 		(fp_text user "${REFERENCE}"
-			(at 0 0 270)
+			(at 0 0 -90)
 			(layer "F.Fab")
 			(effects
@@
 		(tags "SOIC SO")
 		(property "Reference" "U1"
-			(at 0 -3.88 360)
+			(at 0 -3.88 0)
 			(layer "F.SilkS")
 			(effects
@@
 		)
 		(property "Value" "MPXHZ6130"
-			(at 0 3.88 360)
+			(at 0 3.88 0)
 			(layer "F.Fab")
 			(effects
@@
 		)
 		(fp_text user "${REFERENCE}"
-			(at 0 0 360)
+			(at 0 0 0)
 			(layer "F.Fab")
 			(effects
@@
 	)
 	(gr_circle
-		(center 157.433586 95.253248)
-		(end 182.433586 95.253248)
-		(stroke
-			(width 0.25)
-			(type default)
-		)
-		(fill none)
-		(layer "Dwgs.User")
-	)
-	(gr_line
-		(start 132.433586 95.253248)
-		(end 182.433586 95.253248)
-		(stroke
-			(width 0.25)
-			(type default)
-		)
-		(layer "Dwgs.User")
-	)
-	(gr_circle
 		(center 173.343488 111.16315)
 		(end 174.393488 111.16315)
@@
 		(layer "Dwgs.User")
 	)
-	(gr_line
-		(start 175.094118 77.558458)
-		(end 139.592947 112.766432)
-		(stroke
-			(width 0.25)
-			(type default)
-		)
-		(layer "Dwgs.User")
-	)
 	(gr_circle
 		(center 141.523683 79.343345)
@@
 	)
 	(gr_circle
-		(center 157.433586 95.253248)
-		(end 181.433586 95.253248)
-		(stroke
-			(width 0.25)
-			(type default)
-		)
-		(fill none)
-		(layer "Dwgs.User")
-	)
-	(gr_circle
 		(center 141.523683 111.16315)
 		(end 142.573683 111.16315)
@@
 		(layer "Dwgs.User")
 	)
-	(gr_line
-		(start 139.885861 77.446581)
-		(end 175.094118 112.948038)
-		(stroke
-			(width 0.25)
-			(type default)
-		)
-		(layer "Dwgs.User")
-	)
 	(gr_circle
 		(center 173.343488 79.343345)
@@
 		(layer "Dwgs.User")
 	)
-	(gr_line
-		(start 157.433586 70.253248)
-		(end 157.433586 120.253248)
-		(stroke
-			(width 0.25)
-			(type default)
-		)
-		(layer "Dwgs.User")
-	)
 	(gr_circle
 		(center 157.48999 95.19731)
@@
 		(layer "Edge.Cuts")
 	)
+	(gr_text "3.3V\nGND\nSCL\nSDA"
+		(at 148.6 108.3 0)
+		(layer "F.SilkS")
+		(effects
+			(font
+				(size 1 1)
+				(thickness 0.1)
+			)
+			(justify left bottom)
+		)
+	)
+	(gr_text "GND\n"
+		(at 139.1 97.8 0)
+		(layer "F.SilkS")
+		(effects
+			(font
+				(size 1 1)
+				(thickness 0.1)
+			)
+			(justify left bottom)
+		)
+	)
+	(gr_text "5V\n"
+		(at 139 94.1 0)
+		(layer "F.SilkS")
+		(effects
+			(font
+				(size 1 1)
+				(thickness 0.1)
+			)
+			(justify left bottom)
+		)
+	)
+	(gr_text "GND\nSCL\nSDA\nBARO_dev\nBARO_raw"
+		(at 168.7 98 0)
+		(layer "F.SilkS")
+		(effects
+			(font
+				(size 0.75 0.75)
+				(thickness 0.1)
+			)
+			(justify left bottom)
+		)
+	)
 	(segment
 		(start 156.225002 83.974998)
@@
 	)
 	(via
-		(at 165.1 80.5)
+		(at 165.9 79.8)
 		(size 0.6)
 		(drill 0.3)
@@
 	)
 	(via
-		(at 149.86 103.36)
+		(at 149.86 101.6)
 		(size 0.6)
 		(drill 0.3)
@@
 	)
 	(via
-		(at 162.56 93.2)
+		(at 162.9 94.4)
 		(size 0.6)
 		(drill 0.3)
@@
 	)
 	(via
-		(at 149.86 108.44)
+		(at 149.8 109.3)
 		(size 0.6)
 		(drill 0.3)
@@
 	)
 	(via
-		(at 149.86 75.42)
+		(at 148.5 74.9)
 		(size 0.6)
 		(drill 0.3)
@@
 	)
 	(via
-		(at 144.78 85.58)
+		(at 146.3 85.5)
 		(size 0.6)
 		(drill 0.3)
@@
 	)
 	(group ""
-		(members "02dcbc34-d433-4fe0-81d5-dac47c95a433" "1fa984e1-b2e1-4bf6-99f5-85c0a3795c7d"
-			"358e2b99-e86e-4e17-a644-2ef0f2e584fb" "38783365-7eb3-4f54-814a-7da2735f279b"
-			"4bac7c4e-9b57-4931-9602-946633ba3c06" "900db328-0dd7-487f-b113-0d3f4d3b0f8d"
-			"9c98037e-0cc0-46cb-8ff1-f21d4777b062" "c6e8efdd-de69-4e72-9361-4ecb60e1c842"
-			"d298bc4d-3b90-4764-9bf1-44581db4faf2" "e4cb1b2a-b783-454e-9e31-cea177a521f8"
+		(members "358e2b99-e86e-4e17-a644-2ef0f2e584fb" "4bac7c4e-9b57-4931-9602-946633ba3c06"
+			"9c98037e-0cc0-46cb-8ff1-f21d4777b062" "d298bc4d-3b90-4764-9bf1-44581db4faf2"
 		)
 	)
