File: bno_module/bno85/bno85.kicad_pcb (KiCad board)
At the start: 4 copper layers, 50 x 50 mm, 14 parts, among them J1 Conn_01x02_MountingPin, J2 BNO_085, J4 Conn_01x09_MountingPin, U1 AMS1117-3.3

Commit message: final
Other:
- board text added: "5V"
- board text added: "GND"
- board text added: "GND PS0 RST INT MOSI MISO SCK SC PS1"
Changed lines of the file:
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@@
 			(plot_on_all_layers_selection 0x0000000_00000000)
 			(disableapertmacros no)
-			(usegerberextensions no)
-			(usegerberattributes yes)
-			(usegerberadvancedattributes yes)
-			(creategerberjobfile yes)
+			(usegerberextensions yes)
+			(usegerberattributes no)
+			(usegerberadvancedattributes no)
+			(creategerberjobfile no)
 			(dashed_line_dash_ratio 12.000000)
 			(dashed_line_gap_ratio 3.000000)
 			(svgprecision 4)
 			(plotframeref no)
-			(viasonmask no)
+			(viasonmask yes)
 			(mode 1)
 			(useauxorigin no)
@@
 			(psa4output no)
 			(plotreference yes)
-			(plotvalue yes)
+			(plotvalue no)
 			(plotfptext yes)
 			(plotinvisibletext no)
 			(sketchpadsonfab no)
-			(subtractmaskfromsilk no)
+			(subtractmaskfromsilk yes)
 			(outputformat 1)
 			(mirror no)
-			(drillshape 1)
+			(drillshape 0)
 			(scaleselection 1)
-			(outputdirectory "")
+			(outputdirectory "../gerber/")
 		)
 	)
@@
 			(at 0 -3.2 0)
 			(layer "F.SilkS")
+			(hide yes)
 			(effects
 				(font
@@
 		(tags "SOT-363 SC-70-6")
 		(property "Reference" "D1"
-			(at 0 -2.25 270)
+			(at 2.4 0.1 0)
 			(layer "F.SilkS")
 			(effects
@@
 		)
 		(property "Value" " SMF05CT1G"
-			(at 0 2.000001 270)
+			(at 0 2.000001 -90)
 			(layer "F.Fab")
 			(effects
@@
 		)
 		(property "Value" "Conn_01x09_MountingPin"
-			(at 0 3.899999 270)
+			(at 0 3.899999 -90)
 			(layer "F.Fab")
 			(effects
@@
 		)
 		(fp_text user "${REFERENCE}"
-			(at 0 0 270)
+			(at 0 0 -90)
 			(layer "F.Fab")
 			(effects
@@
 		(tags "SOT-363 SC-70-6")
 		(property "Reference" "D2"
-			(at 0 -2.25 360)
+			(at 0 -2.25 0)
 			(layer "F.SilkS")
 			(effects
@@
 		)
 		(property "Value" " SMF05CT1G"
-			(at 0 2.000001 360)
+			(at 0 2.000001 0)
 			(layer "F.Fab")
 			(effects
@@
 		)
 		(property "Value" "AMS1117-3.3"
-			(at 0 4.500001 360)
+			(at 0 4.500001 0)
 			(layer "F.Fab")
 			(effects
@@
 		(tags "Through hole pin header THT 1x10 2.54mm single row")
 		(property "Reference" "J2"
-			(at 0 -2.33 360)
+			(at 0 -2.33 0)
 			(layer "F.SilkS")
 			(hide yes)
@@
 		)
 		(property "Value" "BNO_085"
-			(at 0 25.19 360)
+			(at 0 25.19 0)
 			(layer "F.Fab")
 			(effects
@@
 			(at 0 -3.2 0)
 			(layer "F.SilkS")
+			(hide yes)
 			(effects
 				(font
@@
 		(tags "LED")
 		(property "Reference" "D3"
-			(at 0 1.5 90)
+			(at 2.575001 0.45 90)
 			(layer "F.SilkS")
 			(effects
@@
 			(at 0 -3.899999 90)
 			(layer "F.SilkS")
+			(hide yes)
 			(effects
 				(font
@@
 		(tags "resistor")
 		(property "Reference" "R1"
-			(at 0 1.5 270)
+			(at -2.45 0.1 -90)
 			(layer "F.SilkS")
 			(effects
@@
 		)
 		(property "Value" "2k2"
-			(at 0 1.43 270)
+			(at 0 1.43 -90)
 			(layer "F.Fab")
 			(effects
@@
 		)
 		(fp_text user "${REFERENCE}"
-			(at 0 0 270)
+			(at 0 0 -90)
 			(layer "F.Fab")
 			(effects
@@
 			(at 0 -3.2 0)
 			(layer "F.SilkS")
+			(hide yes)
 			(effects
 				(font
@@
 		(tags "capacitor")
 		(property "Reference" "C1"
-			(at 0 1.700001 360)
+			(at 2.65 0 0)
 			(layer "F.SilkS")
 			(effects
@@
 		)
 		(property "Value" "22uF"
-			(at 0 1.679999 360)
+			(at 0 1.679999 0)
 			(layer "F.Fab")
 			(effects
@@
 		)
 		(fp_text user "${REFERENCE}"
-			(at 0 0 360)
+			(at 0 0 0)
 			(layer "F.Fab")
 			(effects
@@
 			(at 0 -3.2 0)
 			(layer "F.SilkS")
+			(hide yes)
 			(effects
 				(font
@@
 	)
 	(gr_circle
-		(center 207.05 96.7)
-		(end 231.05 96.7)
-		(stroke
-			(width 0.25)
-			(type default)
-		)
-		(fill none)
-		(layer "Dwgs.User")
-	)
-	(gr_circle
 		(center 191.140097 112.609902)
 		(end 192.190097 112.609902)
@@
 		(layer "Dwgs.User")
 	)
-	(gr_line
-		(start 182.05 96.7)
-		(end 232.05 96.7)
-		(stroke
-			(width 0.25)
-			(type default)
-		)
-		(layer "Dwgs.User")
-	)
-	(gr_line
-		(start 224.710532 79.00521)
-		(end 189.209361 114.213184)
-		(stroke
-			(width 0.25)
-			(type default)
-		)
-		(layer "Dwgs.User")
-	)
 	(gr_circle
 		(center 222.959902 112.609902)
@@
 		(layer "Dwgs.User")
 	)
-	(gr_line
-		(start 207.05 71.7)
-		(end 207.05 121.7)
-		(stroke
-			(width 0.25)
-			(type default)
-		)
-		(layer "Dwgs.User")
-	)
-	(gr_line
-		(start 189.502275 78.893333)
-		(end 224.710532 114.39479)
-		(stroke
-			(width 0.25)
-			(type default)
-		)
-		(layer "Dwgs.User")
-	)
-	(gr_circle
-		(center 207.05 96.7)
-		(end 232.05 96.7)
-		(stroke
-			(width 0.25)
-			(type default)
-		)
-		(fill none)
-		(layer "Dwgs.User")
-	)
 	(gr_circle
 		(center 207.05 96.7)
@@
 		(layer "Edge.Cuts")
 	)
+	(gr_text "5V"
+		(at 190.7 95.8 0)
+		(layer "F.SilkS")
+		(effects
+			(font
+				(size 1 1)
+				(thickness 0.1)
+			)
+			(justify left bottom)
+		)
+	)
+	(gr_text "GND\nPS0\nRST\nINT\nMOSI\nMISO\nSCK\nSC\nPS1"
+		(at 215.7 102.1 0)
+		(layer "F.SilkS")
+		(effects
+			(font
+				(size 0.75 0.75)
+				(thickness 0.1)
+			)
+			(justify left bottom)
+		)
+	)
+	(gr_text "GND"
+		(at 190.6 98.3 0)
+		(layer "F.SilkS")
+		(effects
+			(font
+				(size 1 1)
+				(thickness 0.1)
+			)
+			(justify left bottom)
+		)
+	)
 	(segment
 		(start 194.999999 94.525001)
@@
 	)
 	(via
-		(at 216.31 101.48)
+		(at 215 97.6)
 		(size 0.6)
 		(drill 0.3)
@@
 	)
 	(via
-		(at 216.31 98.94)
+		(at 214.4 100.5)
 		(size 0.6)
 		(drill 0.3)
@@
 	)
 	(group ""
-		(members "226c2fa9-91b6-48a0-a128-62bd41e44626" "2c6959e7-2eb2-44c0-ad37-1753dd10bba6"
-			"b6a72528-ebc0-41ca-80a9-c30cf3443461" "c34b30d0-6596-486f-884e-3c199aa9442e"
-			"d0f02753-e79e-4d4d-b76c-b872f3cfbb22" "e3eaab3b-d866-4ebc-8cbf-926d3c3c197e"
-			"e5366b20-61d2-41bf-a0f8-881be9e7684c" "ed245fbe-68a4-4caa-be3d-c9161a4e0cca"
-			"f2469525-3430-46cc-8b44-b5d32c35d740" "ff767000-fdc8-4f52-9756-e80f8eacc790"
+		(members "226c2fa9-91b6-48a0-a128-62bd41e44626" "b6a72528-ebc0-41ca-80a9-c30cf3443461"
+			"e3eaab3b-d866-4ebc-8cbf-926d3c3c197e" "e5366b20-61d2-41bf-a0f8-881be9e7684c"
 		)
 	)
