File: naebsiki/naebsiki.kicad_sch (KiCad schematic)
At the start: 0 parts

Commit message: final
Parts:
- added C1, C2: 15p, Capacitor_SMD:C_0603_1608Metric, symbol BLDC_4-rescue:C-RESCUE-BLDC_4
- added C10, C11, C12, C14, C15, C16, C4, C5, C6, C7, C8, C9: 2.2u, Capacitor_SMD:C_0603_1608Metric, symbol BLDC_4-rescue:C-RESCUE-BLDC_4
- added C13, C3: 100n, Capacitor_SMD:C_0603_1608Metric, symbol BLDC_4-rescue:C-RESCUE-BLDC_4
- added C17: 100n, Capacitor_SMD:C_0402_1005Metric, symbol Device:C_Small
- added C18, C19: 24p, Capacitor_SMD:C_0603_1608Metric, symbol BLDC_4-rescue:C-RESCUE-BLDC_4
- added D1, D2: BLU, LED_SMD:LED_0603_1608Metric, symbol Device:LED
- added H1, H2, H3, H4: MountingHole, MountingHole:MountingHole_2.2mm_M2, symbol Mechanical:MountingHole
- added J1: VIN, Connector_JST:JST_GH_SM02B-GHS-TB_1x02-1MP_P1.25mm_Horizontal, symbol Connector_Generic_MountingPin:Conn_01x02_MountingPin
- added J2: USB_B_Micro, Connector_USB:USB_Mini-B_Lumberg_2486_01_Horizontal, symbol RBoard-rescue:USB_B_Micro-Connector
- added J3: power_jumper, Connector_PinHeader_1.00mm:PinHeader_1x02_P1.00mm_Vertical, symbol Connector_Generic:Conn_01x02
- added J4, J5: PWM, Connector_JST:JST_GH_SM04B-GHS-TB_1x04-1MP_P1.25mm_Horizontal, symbol Connector_Generic_MountingPin:Conn_01x04_MountingPin
- added J6: BNO_MODULE, symbol Connector_Generic_MountingPin:Conn_01x07_MountingPin
- added J7: BAROMODULE, symbol Connector_Generic_MountingPin:Conn_01x03_MountingPin
- added J8: UNUSED, symbol Connector_Generic:Conn_02x07_Counter_Clockwise
- added NTC1: NTC 10k, Resistor_SMD:R_0603_1608Metric, symbol BLDC_4-rescue:R-RESCUE-BLDC_4
- added P1: SWD, Connector_PinHeader_2.54mm:PinHeader_1x05_P2.54mm_Vertical, symbol Connector_Generic:Conn_01x05
- added P2: ST-TF-003A, ST-TF-003A_footprint:SUNTECH_ST-TF-003A, symbol ST-TF-003A:ST-TF-003A
- added R1, R2, R3, R4, R5, R6: 10k, Resistor_SMD:R_0402_1005Metric_Pad0.72x0.64mm_HandSolder, symbol Device:R
- added R10, R11: 10k, Resistor_SMD:R_0402_1005Metric, symbol Device:R_Small
- added R12, R9: 2k2, Resistor_SMD:R_0402_1005Metric_Pad0.72x0.64mm_HandSolder, symbol BLDC_4-rescue:R-RESCUE-BLDC_4
- added R7: 1M, Resistor_SMD:R_0402_1005Metric_Pad0.72x0.64mm_HandSolder, symbol Device:R
- added R8: 10k, Resistor_SMD:R_0402_1005Metric_Pad0.72x0.64mm_HandSolder, symbol BLDC_4-rescue:R-RESCUE-BLDC_4
- added U1: STM32F405RGT6, Package_QFP:LQFP-64_10x10mm_P0.5mm, symbol BLDC_4-rescue:STM32F40X_LQFP64
- added U2: AMS1117-3.3, Package_TO_SOT_SMD:SOT-223-3_TabPin2, symbol Regulator_Linear:AMS1117-3.3
- added U3: W25N01GVZEIG, WinbondFlash:W25N01GVZEIG, symbol RBoard-rescue:W25N01GVZEIG-SchmillipKiCADLibrary
- added X1: 8MHz 10ppm (X50328MSB2GI), Crystal:Crystal_SMD_5032-2Pin_5.0x3.2mm, symbol Device:Crystal_Small
- added Y1: 32.768, Crystal:Crystal_SMD_3215-2Pin_3.2x1.5mm, symbol Device:Crystal
Connections:
- new net: C19.1, U1.3 (PC14-OSC32_IN), Y1.1
- new net: J2.1 (VBUS), J3.2 (Pin_2)
- new net: C2.1, U1.5 (PH0-OSC_IN), X1.1
- new net: D2.2 (A), R12.1
- new net: R12.2, U1.2 (PC13_(RTC_AF1))
- new net: C1.1, U1.6 (PH1-OSC_OUT), X1.2
- new net: C6.1, U1.31 (VCAP1)
- new net: D1.2 (A), R9.1
- new net: C18.1, U1.4 (PC15-OSC32_OUT), Y1.2
- new net: C7.1, U1.47 (VCAP2)
- new net +3V3: C10.2, C11.2, C12.2, C13.1, C15.2, C17.1, C4.2, C5.2, C8.2, C9.2, NTC1.1, P1.1 (Pin_1), P2.4 (VDD), R1.2, R10.1, R11.1, R2.2, R3.2, R4.2, R5.2, R6.2, R9.2, U1.1 (VBAT), U1.13 (VDDA), U1.19 (VDD), U1.32 (VDD), U1.48 (VDD), U1.64 (VDD), U2.2 (VO), U3.8 (VCC)
- new net +5V: C16.2, J1.1 (Pin_1), J3.1 (Pin_1), U2.3 (VI)
- new net BNO_INT: J6.5 (Pin_5), U1.24 (PC4(ADC12_IN14))
- new net BNO_PS0: J6.7 (Pin_7), U1.26 (PB0(ADC12_IN8))
- new net BNO_RST: J6.6 (Pin_6), U1.25 (PC5(ADC12_IN15))
- new net FLASH_!HOLD: R11.2, U1.30 (PB11), U3.7 (~{HOLD})
- new net FLASH_!WP: R10.2, U1.29 (PB10), U3.3 (~{WP})
- new net GND: C1.2, C10.1, C11.1, C12.1, C13.2, C14.2, C15.1, C16.1, C17.2, C18.2, C19.2, C2.2, C3.1, C4.1, C5.1, C6.2, C7.2, C8.1, C9.1, D1.1 (K), D2.1 (K), J1.2 (Pin_2), J1.MP (MountPin), J2.5 (GND), J4.MP (MountPin), J5.MP (MountPin), J6.MP (MountPin), J7.MP (MountPin), P1.3 (Pin_3), P2.6 (VSS), P2.G1 (GND), P2.G2 (GND), P2.G3 (GND), P2.G4 (GND), R7.2, R8.2, U1.12 (VSSA), U1.18 (VSS), U1.60 (BOOT0(VPP)), U1.63 (VSS), U2.1 (GND), U3.4 (GND), U3.9 (EP)
- new net I2C_1_SCL: J7.3 (Pin_3)
- new net I2C_1_SDA: J7.2 (Pin_2)
- new net NRST: C3.2, P1.5 (Pin_5), U1.7 (NRST)
- new net PA8: U1.41 (PA8)
- new net PB1: U1.27 (PB1(ADC12_IN9))
- new net PB2: U1.28 (PB2-BOOT1)
- new net PB3: U1.55 (PB3(JTDO/TRACESWO))
- new net PB5: U1.57 (PB5)
- new net PB7: U1.59 (PB7)
- new net PB9: U1.62 (PB9)
- new net PC0: U1.8 (PC0(ADC123_IN10))
- new net PC1: U1.9 (PC1(ADC123_IN11))
- new net PC2: U1.10 (PC2(ADC123_IN12))
- new net PC3: U1.11 (PC3(ADC123_IN13))
- new net PC6: U1.37 (PC6)
- new net SDIO_CLK: P2.5 (CLK), R6.1, U1.53 (PC12)
- new net SDIO_CMD: P2.3 (CMD), R1.1, U1.54 (PD2)
- new net SDIO_D0: P2.7 (DAT0), R2.1, U1.39 (PC8)
- new net SDIO_D1: P2.8 (DAT1), R3.1, U1.40 (PC9)
- new net SDIO_D2: P2.1 (DAT2), R4.1, U1.51 (PC10)
- new net SDIO_D3: P2.2 (DAT3), R5.1, U1.52 (PC11)
- new net SD_CARD_CD: P2.9 (CD), R7.1, U1.38 (PC7)
- new net SPI2_!CS: U1.33 (PB12), U3.1 (~{CS})
- new net SPI2_MISO: U1.35 (PB14), U3.2 (DO(IO1))
- new net SPI2_MOSI: U1.36 (PB15), U3.5 (DI(IO0))
- new net SPI2_SCK: U1.34 (PB13(OTG_HS_VBUS)), U3.6 (CLK)
- new net SPI_1_CS: J6.1 (Pin_1), U1.20 (PA4(ADC12_IN4/DAC1_OUT))
- new net SPI_1_MISO: J6.3 (Pin_3), U1.22 (PA6(ADC12_IN6))
- new net SPI_1_MOSI: J6.4 (Pin_4), U1.23 (PA7(ADC12_IN7))
- new net SPI_1_SCK: J6.2 (Pin_2), U1.21 (PA5(ADC12_IN5/DAC2_OUT))
- new net SWCLK: P1.2 (Pin_2), U1.49 (PA14(JTCK-SWCLK))
- new net SWDIO: P1.4 (Pin_4), U1.46 (PA13(JTMS-SWDIO))
- new net TEMPERATURE_NTC: C14.1, NTC1.2, R8.1, U1.14 (PA0(ADC123_IN0/WKUP))
- new net TIM1_CH1: J5.1 (Pin_1), U1.61 (PB8)
- new net TIM2_CH1: J5.2 (Pin_2), U1.50 (PA15(JTDI))
- new net TIM3_CH1: J5.3 (Pin_3), U1.56 (PB4(NJTRST))
- new net TIM4_CH1: J5.4 (Pin_4), U1.58 (PB6)
- new net USART_1_RX: J4.2 (Pin_2), U1.43 (PA10)
- new net USART_1_TX: J4.1 (Pin_1), U1.42 (PA9(OTG_FS_VBUS))
- new net USART_2_RX: J4.4 (Pin_4), U1.17 (PA3(ADC123_IN3))
- new net USART_2_TX: J4.3 (Pin_3), U1.16 (PA2(ADC123_IN2))
- new net USB_D+: J2.3 (D+), U1.45 (PA12)
- new net USB_D-: J2.2 (D-), U1.44 (PA11)
- new net baro analog: J7.1 (Pin_1), U1.15 (PA1(ADC123_IN1))
- no-connect marks 0 -> 2
Other:
- removed sheet Barometr
- removed sheet IMU
- removed sheet MCU
- note added: "Bypass, place next to VDD pins"
- note added: "CONNECTORS_BARO"
- note added: "CONNECTORS_BNO"
- note added: "CONNECTORS_UART"
- note added: "FLASH Memory"
- note added: "MOUNTING"
- note added: "POWER_SUPPLY"
- note added: "PWM"
- note added: "Programming / Debug connector"
- note added: "Required for USB to work"
- note added: "Reset pin internally pulled up"
- note added: "SD_CARD_SDIO"
- note added: "TEMP_SENS"
- note added: "USB"
- note added: "or 22pF order both"
