File: 6_layer_MCU/6_layer_MCU.kicad_pcb (KiCad board)
At the start: 6 copper layers, 50 x 50 mm, 74 parts, among them J1 USB_B_Micro, J2 power_jumper, J3 VIN, J5 Conn_02x06_Counter_Clockwise, J6 PWM, J7 PWM, P1 SWD, P2 ST-TF-003A, SW1 SW_SPDT, U1 STM32F405RGT6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

Commit message: final
Parts:
- removed J5: Conn_02x06_Counter_Clockwise, Connector_PinHeader_1.00mm:PinHeader_2x06_P1.00mm_Vertical
- C19, C26, C27, J3, J7, U3: moved to B.Cu
- J1: footprint Connector_USB:USB_Micro-B_Wuerth_629105150521 -> Connector_USB:USB_Mini-B_Lumberg_2486_01_Horizontal; moved to B.Cu
- J2: footprint Connector_PinSocket_2.54mm:PinSocket_1x02_P2.54mm_Vertical -> Connector_PinHeader_1.00mm:PinHeader_1x02_P1.00mm_Vertical
- P1: footprint Connector_PinHeader_2.54mm:PinHeader_1x05_P2.54mm_Vertical -> Connector_PinHeader_1.00mm:PinHeader_1x05_P1.00mm_Vertical
- P2, U4: moved to F.Cu
- R1, R17, R2, R3, R8, R9: footprint Resistor_SMD:R_0603_1608Metric_Pad0.98x0.95mm_HandSolder -> Resistor_SMD:R_0402_1005Metric_Pad0.72x0.64mm_HandSolder
- R10, R11, R12, R13, R14, R15, R16: footprint Resistor_SMD:R_0603_1608Metric_Pad0.98x0.95mm_HandSolder -> Resistor_SMD:R_0402_1005Metric_Pad0.72x0.64mm_HandSolder; moved to B.Cu
- R18, R19, R4, R7: footprint Resistor_SMD:R_0603_1608Metric -> Resistor_SMD:R_0402_1005Metric_Pad0.72x0.64mm_HandSolder
- R5, R6: footprint Resistor_SMD:R_0402_1005Metric -> Resistor_SMD:R_0402_1005Metric_Pad0.72x0.64mm_HandSolder
- moved H4 72.0 mm to (137.0, 85.6)
- moved J1 72.0 mm to (134.5, 100.7)
- moved C16 67.8 mm to (166.9, 93.3), turned to -45 degrees
- moved C15 66.9 mm to (163.8, 81.5), turned to 45 degrees
- moved C6 66.7 mm to (161.4, 88.6), turned to -45 degrees
- moved C17 66.5 mm to (164.6, 91.0), turned to 135 degrees
- moved C1 65.8 mm to (161.7, 94.2), turned to 135 degrees
- moved C7 65.6 mm to (159.1, 86.3), turned to 135 degrees
- moved C8 64.7 mm to (158.4, 89.6), turned to -135 degrees
- moved C3 64.5 mm to (160.4, 98.6), turned to 45 degrees
- moved D3 64.0 mm to (168.9, 113.5), turned to 180 degrees
- moved C13 63.5 mm to (163.3, 105.1), turned to 90 degrees
- moved C27 63.1 mm to (163.1, 122.7), turned to 180 degrees
- moved C26 61.6 mm to (159.9, 122.7)
- moved R19 59.9 mm to (168.6, 112.1)
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Connections:
- C16 pad 2: Net-(C16-Pad2) -> GND
- C17 pad 2: Net-(C16-Pad2) -> GND
- C20 pad 2: Net-(C20-Pad2) -> GND
- C21 pad 2: Net-(C20-Pad2) -> GND
- U1 pad 10: /SPI_2_MISO -> /PB15
- U1 pad 11: /SPI_2_MOSI -> /PB14
- U1 pad 35: /PB14 -> /SPI_2_MISO
- U1 pad 36: /PB15 -> /SPI_2_MOSI
Routing:
- net GND: track 0.00 -> 76.2 mm, vias 0 -> 54
- net +3V3: track 0.00 -> 68.8 mm, vias 0 -> 38
- net +5V: track 0.00 -> 49.4 mm, vias 0 -> 1
- net /FLASH_HOLD: track 0.00 -> 41.0 mm, vias 0 -> 3
- net /BNO_08x_PS0_WEAK: track 0.00 -> 33.4 mm, vias 0 -> 2
- net /TIM1_CH1: track 0.00 -> 32.3 mm, vias 0 -> 4
- net /BAROMETR_OUT: track 0.00 -> 29.7 mm, vias 0 -> 2
- net /BNO_08x_RST: track 0.00 -> 29.1 mm, vias 0 -> 2
- net BOOT0: track 0.00 -> 27.4 mm, vias 0 -> 3
- net /TIM2_CH1: track 0.00 -> 27.1 mm, vias 0 -> 2
- net /BNO_08x_INT: track 0.00 -> 26.3 mm, vias 0 -> 2
- net SWDIO: track 0.00 -> 25.6 mm, vias 0 -> 2
- net NRST: track 0.00 -> 25.5 mm, vias 0 -> 2
- net SWCLK: track 0.00 -> 25.4 mm, vias 0 -> 2
- net USB_D+: track 0.00 -> 21.5 mm, vias 0 -> 1
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- added copper zone on B.Cu, net +3V3
- added copper zone on In3.Cu, net +3V3
- added copper zone on B.Cu, net GND
- added copper zone on F.Cu, net GND
- added copper zone on In1.Cu, net GND
- added copper zone on In4.Cu, net GND

Commit message: update
Parts:
- removed P1: SWD, Connector_PinHeader_1.00mm:PinHeader_1x05_P1.00mm_Vertical
- added J4: Conn_02x03_Counter_Clockwise, Connector_PinHeader_2.54mm:PinHeader_2x03_P2.54mm_Vertical, F.Cu at (133.1, 92.7)
- added R20: 4k7, Resistor_SMD:R_0402_1005Metric_Pad0.72x0.64mm_HandSolder, B.Cu at (142.0, 114.6)
- added R21: 4k7, Resistor_SMD:R_0402_1005Metric_Pad0.72x0.64mm_HandSolder, B.Cu at (143.2, 114.6)
- U5: value BNO055 -> BNO085
Connections:
- U5 pad 10: +3V3 -> GND
- U5 pad 15: GND -> Net-(R20-Pad2)
- U5 pad 16: GND -> Net-(R21-Pad2)
- U5 pad 25: GND -> unconnected-(U5-GNDIO-Pad25)
Routing:
- net Net-(J1-VBUS): track 18.7 -> 26.2 mm
- net Net-(R21-Pad2): track 0.00 -> 7.48 mm, vias 0 -> 1
- net Net-(R20-Pad2): track 0.00 -> 7.17 mm, vias 0 -> 1
- net SWDIO: track 25.6 -> 31.2 mm
- net GND: track 76.2 -> 73.1 mm, vias 54 -> 53
- net +3V3: track 68.8 -> 70.8 mm, vias 38 -> 39
- net NRST: track 25.5 -> 26.6 mm
- net unconnected-(U5-GNDIO-Pad25): track 0.00 -> 0.97 mm, vias 0 -> 1
- net SWCLK: track 25.4 -> 24.8 mm, vias 2 -> 1
- net /BNO_08x_RST: track 29.1 -> 29.6 mm
