File: 6_layer_MCU/6_layer_MCU.kicad_sch (KiCad schematic)
At the start: 74 parts, among them J1 USB_B_Micro, J2 power_jumper, J3 VIN, J5 Conn_02x06_Counter_Clockwise, J6 PWM, J7 PWM, P1 SWD, P2 ST-TF-003A, SW1 SW_SPDT, U1 STM32F405RGT6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

Commit message: final
Parts:
- removed J5: Conn_02x06_Counter_Clockwise, Connector_PinHeader_1.00mm:PinHeader_2x06_P1.00mm_Vertical, symbol Connector_Generic:Conn_02x06_Counter_Clockwise
- J1: footprint Connector_USB:USB_Micro-B_Wuerth_629105150521 -> Connector_USB:USB_Mini-B_Lumberg_2486_01_Horizontal
- J2: footprint Connector_PinSocket_2.54mm:PinSocket_1x02_P2.54mm_Vertical -> Connector_PinHeader_1.00mm:PinHeader_1x02_P1.00mm_Vertical
- P1: footprint Connector_PinHeader_2.54mm:PinHeader_1x05_P2.54mm_Vertical -> Connector_PinHeader_1.00mm:PinHeader_1x05_P1.00mm_Vertical
- R1, R10, R11, R12, R13, R14, R15, R16, R17, R2, R3, R8, R9: footprint Resistor_SMD:R_0603_1608Metric_Pad0.98x0.95mm_HandSolder -> Resistor_SMD:R_0402_1005Metric_Pad0.72x0.64mm_HandSolder
- R18, R19, R4, R7: footprint Resistor_SMD:R_0603_1608Metric -> Resistor_SMD:R_0402_1005Metric_Pad0.72x0.64mm_HandSolder
- R5, R6: footprint Resistor_SMD:R_0402_1005Metric -> Resistor_SMD:R_0402_1005Metric_Pad0.72x0.64mm_HandSolder
Connections:
- net GND: now also C16.2, C17.2, C20.2, C21.2
- net PB14: now also U1.11 (PC3(ADC123_IN13)); no longer U1.35 (PB14)
- net PB15: now also U1.10 (PC2(ADC123_IN12)); no longer U1.36 (PB15)
- net SPI_2_MISO: now also U1.35 (PB14); no longer U1.10 (PC2(ADC123_IN12))
- net SPI_2_MOSI: now also U1.36 (PB15); no longer U1.11 (PC3(ADC123_IN13))
- no-connect marks 3 -> 2
Other:
- title: (none) -> Брекешев Бактияр 

Commit message: update
Parts:
- removed P1: SWD, Connector_PinHeader_1.00mm:PinHeader_1x05_P1.00mm_Vertical, symbol Connector_Generic:Conn_01x05
- added J4: Conn_02x03_Counter_Clockwise, Connector_PinHeader_2.54mm:PinHeader_2x03_P2.54mm_Vertical, symbol Connector_Generic:Conn_02x03_Counter_Clockwise
- added R20, R21: 4k7, Resistor_SMD:R_0402_1005Metric_Pad0.72x0.64mm_HandSolder, symbol Device:R
- U5: value BNO055 -> BNO085
Connections:
- net +3V3: now also J4.3 (Pin_3), R20.1, R21.1; no longer U5.10 (BL_IND)
- net GND: now also U5.10 (BL_IND), J4.2 (Pin_2), J4.6 (Pin_6); no longer U5.15 (GNDIO), U5.16 (GNDIO), U5.25 (GNDIO)
- net NRST: now also J4.5 (Pin_5)
- net SWCLK: now also J4.4 (Pin_4)
- net SWDIO: now also J4.1 (Pin_1)
- new net: R20.2, U5.15 (GNDIO)
- new net: R21.2, U5.16 (GNDIO)
